File: MakeItRain/MakeItRain.kicad_pcb (KiCad board)
At the start: 4 copper layers, 151.1 x 71.1 mm, 68 parts, among them IC1 OPA2340PA, IC2 LM2597MX-5.0_NOPB, J1 Conn_02x16_Odd_Even, J2 Conn_02x19_Odd_Even, J3 Conn_01x19, P1 Screw_Terminal_01x02, Q1 IRF9Z34NPBF, Q10 IRF9Z34NPBF, Q11 2N7000, Q12 2N7000, Q13 IRF9Z34NPBF, Q2 2N7000, Q3 2N7000, Q4 IRF9Z34NPBF, Q5 2N7000, Q6 2N7000, Q7 IRF9Z34NPBF, Q8 2N7000, Q9 2N7000, U1 178.6165.0001

Commit message: wip for hardware
Parts:
- removed R18, R23: 1M, Resistor_THT:R_Axial_DIN0207_L6.3mm_D2.5mm_P2.54mm_Vertical
- added C9: 0.1uF, Capacitor_THT:C_Rect_L9.0mm_W3.6mm_P7.50mm_MKT, F.Cu at (140.3, 114.3)
- added D2: 1N4007, Diode_THT:D_DO-41_SOD81_P10.16mm_Horizontal, F.Cu at (61.4, 104.1)
- added D4: 1N4007, Diode_THT:D_DO-41_SOD81_P10.16mm_Horizontal, F.Cu at (61.2, 108.9)
- added D6: 1N4007, Diode_THT:D_DO-41_SOD81_P10.16mm_Horizontal, F.Cu at (75.5, 104.3)
- added D8: 1N4007, Diode_THT:D_DO-41_SOD81_P10.16mm_Horizontal, F.Cu at (89.4, 104.3)
- added IC3: SN7404DR, SamacSys_Parts:SOIC127P600X175-14N, B.Cu at (118.9, 101.6)
- added IC4: LM2597MX-5.0_NOPB, SamacSys_Parts:SOIC127P600X175-8N, F.Cu at (53.3, 91.5)
- added IC5: OPA2340PA, SamacSys_Parts:DIP794W53P254L959H508Q8N, F.Cu at (144.0, 106.3)
- added U2: S8411-45R, SamacSys_Parts:S8411-45R_1, F.Cu at (162.3, 109.6)
- IC1: value OPA2340PA -> DS3231SN#; footprint SamacSys_Parts:DIP794W53P254L959H508Q8N -> SamacSys_Parts:SOIC127P1032X265-16N; moved to B.Cu
- IC2: value LM2597MX-5.0_NOPB -> LTV-846S; footprint SamacSys_Parts:SOIC127P600X175-8N -> SamacSys_Parts:SOP254P1016X460-16N; moved to B.Cu
- R13: value 1M -> 47k; footprint Resistor_THT:R_Axial_DIN0207_L6.3mm_D2.5mm_P2.54mm_Vertical -> Resistor_THT:R_Axial_DIN0207_L6.3mm_D2.5mm_P5.08mm_Vertical
- R3: value 120k -> 10k; footprint Resistor_THT:R_Axial_DIN0207_L6.3mm_D2.5mm_P5.08mm_Vertical -> Resistor_THT:R_Axial_DIN0207_L6.3mm_D2.5mm_P2.54mm_Vertical
- R4: value 15k -> 10k; footprint Resistor_THT:R_Axial_DIN0207_L6.3mm_D2.5mm_P5.08mm_Vertical -> Resistor_THT:R_Axial_DIN0207_L6.3mm_D2.5mm_P2.54mm_Vertical
- R5: value 47k -> 120k
- R8: value 1M -> 15k; footprint Resistor_THT:R_Axial_DIN0207_L6.3mm_D2.5mm_P2.54mm_Vertical -> Resistor_THT:R_Axial_DIN0207_L6.3mm_D2.5mm_P5.08mm_Vertical
- moved IC2 47.3 mm to (95.6, 112.5), turned to 90 degrees
- moved IC1 18.2 mm to (161.5, 110.9), turned to 180 degrees
- moved R4 3.80 mm to (160.6, 100.4)
- moved R5 2.45 mm to (151.8, 101.8)
- moved R2 1.95 mm to (151.7, 97.2)
- moved R3 1.95 mm to (160.6, 97.2)
Connections:
- net /P23 renamed /Zone4IO/ZoneOutputTTL
- IC1 pad 1: /D4 -> unconnected-(IC1-Pad1)
- IC1 pad 2: /D4 -> +3V3
- IC1 pad 3: Net-(IC1-Pad3) -> unconnected-(IC1-Pad3)
- IC1 pad 4: GND -> unconnected-(IC1-Pad4)
- IC1 pad 5: (no net) -> GND
- IC1 pad 6: (no net) -> GND
- IC1 pad 7: (no net) -> GND
- IC1 pad 8: +3V3 -> GND
- IC2 pad 1: Net-(IC2-Pad1) -> unconnected-(IC2-Pad1)
- IC2 pad 2: Net-(C1-Pad1) -> unconnected-(IC2-Pad2)
- IC2 pad 3: +5V -> unconnected-(IC2-Pad3)
- IC2 pad 4: +5V -> unconnected-(IC2-Pad4)
- IC2 pad 5: Net-(C2-Pad1) -> unconnected-(IC2-Pad5)
- IC2 pad 6: GND -> unconnected-(IC2-Pad6)
- IC2 pad 7: +VDC -> unconnected-(IC2-Pad7)
- IC2 pad 8: Net-(D1-Pad1) -> unconnected-(IC2-Pad8)
- J2 pad 35: (no net) -> unconnected-(J2-Pad35)
- J2 pad 36: (no net) -> unconnected-(J2-Pad36)
- J3 pad 13: /D4 -> unconnected-(J3-Pad13)
- J3 pad 17: (no net) -> /SD1
- J3 pad 18: (no net) -> /SDD
- J3 pad 19: (no net) -> /CLK
- Q11 pad 1: /D34 -> GND
- Q11 pad 3: +3V3 -> Net-(Q11-Pad3)
- Q12 pad 2: /D12 -> /Zone3IO/ZoneOutputTTL
- Q2 pad 1: /SVP -> GND
- Q2 pad 3: +3V3 -> Net-(Q2-Pad3)
- Q3 pad 2: /D27 -> /Zone1IO/ZoneOutputTTL
- Q5 pad 1: /SVN -> GND
- Q5 pad 3: +3V3 -> Net-(Q5-Pad3)
- Q6 pad 2: /D14 -> /Zone2IO/ZoneOutputTTL
- Q8 pad 1: /D35 -> GND
- Q8 pad 3: +3V3 -> Net-(Q8-Pad3)
- R13 pad 1: /SVN -> Net-(IC5-Pad1)
- R14 pad 1: /D14 -> /Zone2IO/ZoneOutputTTL
- R24 pad 1: /D12 -> /Zone3IO/ZoneOutputTTL
- R3 pad 1: +VDC -> +3V3
- R3 pad 2: Net-(IC1-Pad3) -> /SCL
- R4 pad 1: Net-(IC1-Pad3) -> +3V3
- R4 pad 2: GND -> /SDA
- R5 pad 1: /D4 -> +VDC
- R5 pad 2: GND -> Net-(IC5-Pad3)
- R6 pad 2: Net-(IC2-Pad1) -> Net-(IC4-Pad1)
- R8 pad 1: /SVP -> Net-(IC5-Pad3)
- R9 pad 1: /D27 -> /Zone1IO/ZoneOutputTTL
Routing:
- net +3V3: track 171.1 -> 0.00 mm
- net /D35: track 124.8 -> 0.00 mm
- net GND: track 311.7 -> 206.3 mm, vias 1 -> 0
- net /D21: track 104.0 -> 0.00 mm
- net /D22: track 102.6 -> 0.00 mm
- net /D32: track 92.4 -> 0.00 mm
- net /RX: track 87.2 -> 0.00 mm, vias 1 -> 0
- net /TX: track 87.1 -> 0.00 mm, vias 1 -> 0
- net /D2: track 83.8 -> 0.00 mm
- net /D33: track 81.9 -> 0.00 mm
- net /D23: track 80.9 -> 0.00 mm
- net /D19: track 80.0 -> 0.00 mm, vias 1 -> 0
- net /D34: track 78.3 -> 0.00 mm, vias 1 -> 0
- net /D4: track 77.5 -> 0.00 mm
- net /D17: track 74.6 -> 0.00 mm, vias 1 -> 0
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Other:
- board text added: "MakeItRain V0.3"
- board text removed: "MakeItRain V0.2"
