File: MakeItRain/file61506092.kicad_sch (KiCad schematic)
At the start: 10 parts, among them Q2 2N7000, Q3 2N7000, Q4 IRF9Z34NPBF

Commit message: wip for hardware
Parts:
- added D4: 1N4007, Diode_THT:D_DO-41_SOD81_P10.16mm_Horizontal, symbol Diode:1N4007
- renumbered C5 to C6, D3 to D5, Q2 to Q5, Q3 to Q6, Q4 to Q7, R7 to R12, R9 to R14, R10 to R15, R11 to R16, Z5 to Z6
Connections:
- net ZoneInputTTL: now also D4.2 (A); no longer Q5.3 (D)
- new net: D4.1 (K), Q5.3 (D)
Changed lines of the file:
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@@
-    (stroke (width 0) (type default) (color 0 0 0 0))
-  )
-  (wire (pts (xy 62.23 71.12) (xy 62.23 66.04))
     (stroke (width 0) (type default) (color 0 0 0 0))
   )
@@
     (stroke (width 0) (type default) (color 0 0 0 0))
   )
+  (wire (pts (xy 62.23 63.5) (xy 62.23 71.12))
+    (stroke (width 0) (type default) (color 0 0 0 0))
+  )
   (wire (pts (xy 125.73 125.73) (xy 125.73 121.92))
     (stroke (width 0) (type default) (color 0 0 0 0))
@@
     (stroke (width 0) (type default) (color 0 0 0 0))
   )
+  (wire (pts (xy 76.2 63.5) (xy 77.47 63.5))
+    (stroke (width 0) (type default) (color 0 0 0 0))
+  )
   (wire (pts (xy 118.11 121.92) (xy 125.73 121.92))
+    (stroke (width 0) (type default) (color 0 0 0 0))
+  )
+  (wire (pts (xy 68.58 63.5) (xy 62.23 63.5))
     (stroke (width 0) (type default) (color 0 0 0 0))
   )
@@
     (effects (font (size 1.27 1.27)) (justify left))
   )
-  (hierarchical_label "ZoneInputTTL" (shape input) (at 62.23 66.04 0)
+  (hierarchical_label "ZoneInputTTL" (shape input) (at 77.47 63.5 0)
     (effects (font (size 1.27 1.27)) (justify left))
   )
@@
   (symbol (lib_id "Transistor_FET:2N7000") (at 59.69 76.2 0)
     (in_bom yes) (on_board yes)
-    (property "Reference" "Q2" (id 0) (at 64.8716 75.0316 0)
+    (property "Reference" "Q5" (id 0) (at 64.8716 75.0316 0)
       (effects (font (size 1.27 1.27)) (justify left))
     )
@@
   (symbol (lib_id "Device:R") (at 54.61 83.82 0)
     (in_bom yes) (on_board yes)
-    (property "Reference" "R7" (id 0) (at 56.388 82.6516 0)
+    (property "Reference" "R12" (id 0) (at 56.388 82.6516 0)
       (effects (font (size 1.27 1.27)) (justify left))
     )
@@
   (symbol (lib_id "power:GND") (at 62.23 96.52 0)
     (in_bom yes) (on_board yes)
-    (property "Reference" "#PWR028" (id 0) (at 62.23 102.87 0)
+    (property "Reference" "#PWR032" (id 0) (at 62.23 102.87 0)
       (effects (font (size 1.27 1.27)) hide)
     )
@@
   (symbol (lib_id "Transistor_FET:2N7000") (at 123.19 105.41 0)
     (in_bom yes) (on_board yes)
-    (property "Reference" "Q3" (id 0) (at 128.3716 104.2416 0)
+    (property "Reference" "Q6" (id 0) (at 128.3716 104.2416 0)
       (effects (font (size 1.27 1.27)) (justify left))
     )
@@
   (symbol (lib_id "Device:R") (at 118.11 118.11 0)
     (in_bom yes) (on_board yes)
-    (property "Reference" "R9" (id 0) (at 119.888 116.9416 0)
+    (property "Reference" "R14" (id 0) (at 119.888 116.9416 0)
       (effects (font (size 1.27 1.27)) (justify left))
     )
@@
   (symbol (lib_id "power:GND") (at 125.73 125.73 0)
     (in_bom yes) (on_board yes)
-    (property "Reference" "#PWR029" (id 0) (at 125.73 132.08 0)
+    (property "Reference" "#PWR033" (id 0) (at 125.73 132.08 0)
       (effects (font (size 1.27 1.27)) hide)
     )
@@
   (symbol (lib_id "Device:R") (at 125.73 91.44 0)
     (in_bom yes) (on_board yes)
-    (property "Reference" "R11" (id 0) (at 127.508 90.2716 0)
+    (property "Reference" "R16" (id 0) (at 127.508 90.2716 0)
       (effects (font (size 1.27 1.27)) (justify left))
     )
@@
   (symbol (lib_id "Device:R") (at 125.73 78.74 0)
     (in_bom yes) (on_board yes)
-    (property "Reference" "R10" (id 0) (at 127.508 77.5716 0)
+    (property "Reference" "R15" (id 0) (at 127.508 77.5716 0)
       (effects (font (size 1.27 1.27)) (justify left))
     )
@@
   (symbol (lib_id "SamacSys_Parts:IRF9Z34NPBF") (at 138.43 85.09 0)
     (in_bom yes) (on_board yes)
-    (property "Reference" "Q4" (id 0) (at 149.352 81.3816 0)
+    (property "Reference" "Q7" (id 0) (at 149.352 81.3816 0)
       (effects (font (size 1.27 1.27)) (justify left))
     )
@@
   (symbol (lib_id "power:+VDC") (at 135.89 55.88 0)
     (in_bom yes) (on_board yes)
-    (property "Reference" "#PWR030" (id 0) (at 135.89 58.42 0)
+    (property "Reference" "#PWR034" (id 0) (at 135.89 58.42 0)
       (effects (font (size 1.27 1.27)) hide)
     )
@@
   (symbol (lib_id "Device:D_Schottky") (at 142.24 101.6 270)
     (in_bom yes) (on_board yes)
-    (property "Reference" "D3" (id 0) (at 144.272 100.4316 90)
+    (property "Reference" "D5" (id 0) (at 144.272 100.4316 90)
       (effects (font (size 1.27 1.27)) (justify left))
     )
@@
   (symbol (lib_id "SamacSys_Parts:BZX79C10") (at 135.89 62.23 90) (mirror x)
     (in_bom yes) (on_board yes)
-    (property "Reference" "Z5" (id 0) (at 139.192 68.6816 90)
+    (property "Reference" "Z6" (id 0) (at 139.192 68.6816 90)
       (effects (font (size 1.27 1.27)) (justify right))
     )
@@
   (symbol (lib_id "Device:C") (at 44.45 83.82 0)
     (in_bom yes) (on_board yes)
-    (property "Reference" "C5" (id 0) (at 47.371 82.6516 0)
+    (property "Reference" "C6" (id 0) (at 47.371 82.6516 0)
       (effects (font (size 1.27 1.27)) (justify left))
     )
@@
       (effects (font (size 1.27 1.27)) hide)
     )
+    (pin "1")
+    (pin "2")
+  )
+  (symbol (lib_id "Diode:1N4007") (at 72.39 63.5 0)
+    (in_bom yes) (on_board yes)
+    (property "Reference" "D4" (id 0) (at 68.58 60.8035 0))
+    (property "Value" "1N4007" (id 1) (at 72.39 61.0386 0))
+    (property "Footprint" "Diode_THT:D_DO-41_SOD81_P10.16mm_Horizontal" (id 2) (at 72.39 67.945 0)
+      (effects (font (size 1.27 1.27)) hide)
+    )
+    (property "Datasheet" "http://www.vishay.com/docs/88503/1n4001.pdf" (id 3) (at 72.39 63.5 0)
+      (effects (font (size 1.27 1.27)) hide)
+    )

Commit message: wip
Parts:
- renumbered C6 to C7, D5 to D7, D4 to D8, Q7 to Q10, Q5 to Q8, Q6 to Q9, R12 to R17, R14 to R19, R15 to R20, R16 to R21, Z6 to Z7
Changed lines of the file:
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@@
   (symbol (lib_id "Transistor_FET:2N7000") (at 59.69 76.2 0)
     (in_bom yes) (on_board yes)
-    (property "Reference" "Q5" (id 0) (at 64.8716 75.0316 0)
+    (property "Reference" "Q8" (id 0) (at 64.8716 75.0316 0)
       (effects (font (size 1.27 1.27)) (justify left))
     )
@@
   (symbol (lib_id "Device:R") (at 54.61 83.82 0)
     (in_bom yes) (on_board yes)
-    (property "Reference" "R12" (id 0) (at 56.388 82.6516 0)
+    (property "Reference" "R17" (id 0) (at 56.388 82.6516 0)
       (effects (font (size 1.27 1.27)) (justify left))
     )
@@
   (symbol (lib_id "power:GND") (at 62.23 96.52 0)
     (in_bom yes) (on_board yes)
-    (property "Reference" "#PWR032" (id 0) (at 62.23 102.87 0)
+    (property "Reference" "#PWR036" (id 0) (at 62.23 102.87 0)
       (effects (font (size 1.27 1.27)) hide)
     )
@@
   (symbol (lib_id "Transistor_FET:2N7000") (at 123.19 105.41 0)
     (in_bom yes) (on_board yes)
-    (property "Reference" "Q6" (id 0) (at 128.3716 104.2416 0)
+    (property "Reference" "Q9" (id 0) (at 128.3716 104.2416 0)
       (effects (font (size 1.27 1.27)) (justify left))
     )
@@
   (symbol (lib_id "Device:R") (at 118.11 118.11 0)
     (in_bom yes) (on_board yes)
-    (property "Reference" "R14" (id 0) (at 119.888 116.9416 0)
+    (property "Reference" "R19" (id 0) (at 119.888 116.9416 0)
       (effects (font (size 1.27 1.27)) (justify left))
     )
@@
   (symbol (lib_id "power:GND") (at 125.73 125.73 0)
     (in_bom yes) (on_board yes)
-    (property "Reference" "#PWR033" (id 0) (at 125.73 132.08 0)
+    (property "Reference" "#PWR037" (id 0) (at 125.73 132.08 0)
       (effects (font (size 1.27 1.27)) hide)
     )
@@
   (symbol (lib_id "Device:R") (at 125.73 91.44 0)
     (in_bom yes) (on_board yes)
-    (property "Reference" "R16" (id 0) (at 127.508 90.2716 0)
+    (property "Reference" "R21" (id 0) (at 127.508 90.2716 0)
       (effects (font (size 1.27 1.27)) (justify left))
     )
@@
   (symbol (lib_id "Device:R") (at 125.73 78.74 0)
     (in_bom yes) (on_board yes)
-    (property "Reference" "R15" (id 0) (at 127.508 77.5716 0)
+    (property "Reference" "R20" (id 0) (at 127.508 77.5716 0)
       (effects (font (size 1.27 1.27)) (justify left))
     )
@@
   (symbol (lib_id "SamacSys_Parts:IRF9Z34NPBF") (at 138.43 85.09 0)
     (in_bom yes) (on_board yes)
-    (property "Reference" "Q7" (id 0) (at 149.352 81.3816 0)
+    (property "Reference" "Q10" (id 0) (at 149.352 81.3816 0)
       (effects (font (size 1.27 1.27)) (justify left))
     )
@@
   (symbol (lib_id "power:+VDC") (at 135.89 55.88 0)
     (in_bom yes) (on_board yes)
-    (property "Reference" "#PWR034" (id 0) (at 135.89 58.42 0)
+    (property "Reference" "#PWR038" (id 0) (at 135.89 58.42 0)
       (effects (font (size 1.27 1.27)) hide)
     )
@@
   (symbol (lib_id "Device:D_Schottky") (at 142.24 101.6 270)
     (in_bom yes) (on_board yes)
-    (property "Reference" "D5" (id 0) (at 144.272 100.4316 90)
+    (property "Reference" "D7" (id 0) (at 144.272 100.4316 90)
       (effects (font (size 1.27 1.27)) (justify left))
     )
@@
   (symbol (lib_id "SamacSys_Parts:BZX79C10") (at 135.89 62.23 90) (mirror x)
     (in_bom yes) (on_board yes)
-    (property "Reference" "Z6" (id 0) (at 139.192 68.6816 90)
+    (property "Reference" "Z7" (id 0) (at 139.192 68.6816 90)
       (effects (font (size 1.27 1.27)) (justify right))
     )
@@
   (symbol (lib_id "Device:C") (at 44.45 83.82 0)
     (in_bom yes) (on_board yes)
-    (property "Reference" "C6" (id 0) (at 47.371 82.6516 0)
+    (property "Reference" "C7" (id 0) (at 47.371 82.6516 0)
       (effects (font (size 1.27 1.27)) (justify left))
     )
@@
   (symbol (lib_id "Diode:1N4007") (at 72.39 63.5 0)
     (in_bom yes) (on_board yes)
-    (property "Reference" "D4" (id 0) (at 68.58 60.8035 0))
+    (property "Reference" "D8" (id 0) (at 68.58 60.8035 0))
     (property "Value" "1N4007" (id 1) (at 72.39 61.0386 0))
     (property "Footprint" "Diode_THT:D_DO-41_SOD81_P10.16mm_Horizontal" (id 2) (at 72.39 67.945 0)

Commit message: wip for input fix.
Parts:
- renumbered C7 to C5, D8 to D7, D7 to D8, Q8 to Q10, Q9 to Q11, Q10 to Q12, R17 to R15, R19 to R16, R20 to R17, R21 to R18, Z7 to Z8
Changed lines of the file:
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@@
   (symbol (lib_id "Transistor_FET:2N7000") (at 59.69 76.2 0)
     (in_bom yes) (on_board yes)
-    (property "Reference" "Q8" (id 0) (at 64.8716 75.0316 0)
+    (property "Reference" "Q10" (id 0) (at 64.8716 75.0316 0)
       (effects (font (size 1.27 1.27)) (justify left))
     )
@@
   (symbol (lib_id "Device:R") (at 54.61 83.82 0)
     (in_bom yes) (on_board yes)
-    (property "Reference" "R17" (id 0) (at 56.388 82.6516 0)
+    (property "Reference" "R15" (id 0) (at 56.388 82.6516 0)
       (effects (font (size 1.27 1.27)) (justify left))
     )
@@
   (symbol (lib_id "power:GND") (at 62.23 96.52 0)
     (in_bom yes) (on_board yes)
-    (property "Reference" "#PWR036" (id 0) (at 62.23 102.87 0)
+    (property "Reference" "#PWR028" (id 0) (at 62.23 102.87 0)
       (effects (font (size 1.27 1.27)) hide)
     )
@@
   (symbol (lib_id "Transistor_FET:2N7000") (at 123.19 105.41 0)
     (in_bom yes) (on_board yes)
-    (property "Reference" "Q9" (id 0) (at 128.3716 104.2416 0)
+    (property "Reference" "Q11" (id 0) (at 128.3716 104.2416 0)
       (effects (font (size 1.27 1.27)) (justify left))
     )
@@
   (symbol (lib_id "Device:R") (at 118.11 118.11 0)
     (in_bom yes) (on_board yes)
-    (property "Reference" "R19" (id 0) (at 119.888 116.9416 0)
+    (property "Reference" "R16" (id 0) (at 119.888 116.9416 0)
       (effects (font (size 1.27 1.27)) (justify left))
     )
@@
   (symbol (lib_id "power:GND") (at 125.73 125.73 0)
     (in_bom yes) (on_board yes)
-    (property "Reference" "#PWR037" (id 0) (at 125.73 132.08 0)
+    (property "Reference" "#PWR029" (id 0) (at 125.73 132.08 0)
       (effects (font (size 1.27 1.27)) hide)
     )
@@
   (symbol (lib_id "Device:R") (at 125.73 91.44 0)
     (in_bom yes) (on_board yes)
-    (property "Reference" "R21" (id 0) (at 127.508 90.2716 0)
+    (property "Reference" "R18" (id 0) (at 127.508 90.2716 0)
       (effects (font (size 1.27 1.27)) (justify left))
     )
@@
   (symbol (lib_id "Device:R") (at 125.73 78.74 0)
     (in_bom yes) (on_board yes)
-    (property "Reference" "R20" (id 0) (at 127.508 77.5716 0)
+    (property "Reference" "R17" (id 0) (at 127.508 77.5716 0)
       (effects (font (size 1.27 1.27)) (justify left))
     )
@@
   (symbol (lib_id "SamacSys_Parts:IRF9Z34NPBF") (at 138.43 85.09 0)
     (in_bom yes) (on_board yes)
-    (property "Reference" "Q10" (id 0) (at 149.352 81.3816 0)
+    (property "Reference" "Q12" (id 0) (at 149.352 81.3816 0)
       (effects (font (size 1.27 1.27)) (justify left))
     )
@@
   (symbol (lib_id "power:+VDC") (at 135.89 55.88 0)
     (in_bom yes) (on_board yes)
-    (property "Reference" "#PWR038" (id 0) (at 135.89 58.42 0)
+    (property "Reference" "#PWR030" (id 0) (at 135.89 58.42 0)
       (effects (font (size 1.27 1.27)) hide)
     )
@@
   (symbol (lib_id "Device:D_Schottky") (at 142.24 101.6 270)
     (in_bom yes) (on_board yes)
-    (property "Reference" "D7" (id 0) (at 144.272 100.4316 90)
+    (property "Reference" "D8" (id 0) (at 144.272 100.4316 90)
       (effects (font (size 1.27 1.27)) (justify left))
     )
@@
   (symbol (lib_id "SamacSys_Parts:BZX79C10") (at 135.89 62.23 90) (mirror x)
     (in_bom yes) (on_board yes)
-    (property "Reference" "Z7" (id 0) (at 139.192 68.6816 90)
+    (property "Reference" "Z8" (id 0) (at 139.192 68.6816 90)
       (effects (font (size 1.27 1.27)) (justify right))
     )
@@
   (symbol (lib_id "Device:C") (at 44.45 83.82 0)
     (in_bom yes) (on_board yes)
-    (property "Reference" "C7" (id 0) (at 47.371 82.6516 0)
+    (property "Reference" "C5" (id 0) (at 47.371 82.6516 0)
       (effects (font (size 1.27 1.27)) (justify left))
     )
@@
   (symbol (lib_id "Diode:1N4007") (at 72.39 63.5 0)
     (in_bom yes) (on_board yes)
-    (property "Reference" "D8" (id 0) (at 68.58 60.8035 0))
+    (property "Reference" "D7" (id 0) (at 68.58 60.8035 0))
     (property "Value" "1N4007" (id 1) (at 72.39 61.0386 0))
     (property "Footprint" "Diode_THT:D_DO-41_SOD81_P10.16mm_Horizontal" (id 2) (at 72.39 67.945 0)

Commit message: wip for layout
Parts:
- renumbered D7 to D8, D8 to D9, R15 to R17, R16 to R18, R17 to R19, R18 to R20
Changed lines of the file:
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@@
   (symbol (lib_id "Device:R") (at 54.61 83.82 0)
     (in_bom yes) (on_board yes)
-    (property "Reference" "R15" (id 0) (at 56.388 82.6516 0)
+    (property "Reference" "R17" (id 0) (at 56.388 82.6516 0)
       (effects (font (size 1.27 1.27)) (justify left))
     )
@@
   (symbol (lib_id "power:GND") (at 62.23 96.52 0)
     (in_bom yes) (on_board yes)
-    (property "Reference" "#PWR028" (id 0) (at 62.23 102.87 0)
+    (property "Reference" "#PWR031" (id 0) (at 62.23 102.87 0)
       (effects (font (size 1.27 1.27)) hide)
     )
@@
   (symbol (lib_id "Device:R") (at 118.11 118.11 0)
     (in_bom yes) (on_board yes)
-    (property "Reference" "R16" (id 0) (at 119.888 116.9416 0)
+    (property "Reference" "R18" (id 0) (at 119.888 116.9416 0)
       (effects (font (size 1.27 1.27)) (justify left))
     )
@@
   (symbol (lib_id "power:GND") (at 125.73 125.73 0)
     (in_bom yes) (on_board yes)
-    (property "Reference" "#PWR029" (id 0) (at 125.73 132.08 0)
+    (property "Reference" "#PWR032" (id 0) (at 125.73 132.08 0)
       (effects (font (size 1.27 1.27)) hide)
     )
@@
   (symbol (lib_id "Device:R") (at 125.73 91.44 0)
     (in_bom yes) (on_board yes)
-    (property "Reference" "R18" (id 0) (at 127.508 90.2716 0)
+    (property "Reference" "R20" (id 0) (at 127.508 90.2716 0)
       (effects (font (size 1.27 1.27)) (justify left))
     )
@@
   (symbol (lib_id "Device:R") (at 125.73 78.74 0)
     (in_bom yes) (on_board yes)
-    (property "Reference" "R17" (id 0) (at 127.508 77.5716 0)
+    (property "Reference" "R19" (id 0) (at 127.508 77.5716 0)
       (effects (font (size 1.27 1.27)) (justify left))
     )
@@
   (symbol (lib_id "power:+VDC") (at 135.89 55.88 0)
     (in_bom yes) (on_board yes)
-    (property "Reference" "#PWR030" (id 0) (at 135.89 58.42 0)
+    (property "Reference" "#PWR033" (id 0) (at 135.89 58.42 0)
       (effects (font (size 1.27 1.27)) hide)
     )
@@
   (symbol (lib_id "Device:D_Schottky") (at 142.24 101.6 270)
     (in_bom yes) (on_board yes)
-    (property "Reference" "D8" (id 0) (at 144.272 100.4316 90)
+    (property "Reference" "D9" (id 0) (at 144.272 100.4316 90)
       (effects (font (size 1.27 1.27)) (justify left))
     )
@@
   (symbol (lib_id "Diode:1N4007") (at 72.39 63.5 0)
     (in_bom yes) (on_board yes)
-    (property "Reference" "D7" (id 0) (at 68.58 60.8035 0))
+    (property "Reference" "D8" (id 0) (at 68.58 60.8035 0))
     (property "Value" "1N4007" (id 1) (at 72.39 61.0386 0))
     (property "Footprint" "Diode_THT:D_DO-41_SOD81_P10.16mm_Horizontal" (id 2) (at 72.39 67.945 0)

Commit message: pre routing
Parts:
- renumbered D9 to D7
Changed lines of the file:
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@@
   (symbol (lib_id "Device:D_Schottky") (at 142.24 101.6 270)
     (in_bom yes) (on_board yes)
-    (property "Reference" "D9" (id 0) (at 144.272 100.4316 90)
+    (property "Reference" "D7" (id 0) (at 144.272 100.4316 90)
       (effects (font (size 1.27 1.27)) (justify left))
     )
